Commit message: change cyberdog_description to xpp_cyberdog

File: robots/xpp_cyberdog/urdf/cyberdog_description.urdf (robot description, URDF)
Before this commit: robot cyberdog_description, 19 links, 18 joints
Links:
- link FL_calf: geometry collision mesh filename=package://xpp_cyberdog/meshes/link_knee_fl.STL; visual mesh filename=package://xpp_cyberdog/meshes/link_knee_fl.STL
- link FL_hip: geometry collision mesh filename=package://xpp_cyberdog/meshes/link_abad_fl.STL; visual mesh filename=package://xpp_cyberdog/meshes/link_abad_fl.STL
- link FL_thigh: geometry collision mesh filename=package://xpp_cyberdog/meshes/link_hip_fl.STL; visual mesh filename=package://xpp_cyberdog/meshes/link_hip_fl.STL
- link FR_calf: geometry collision mesh filename=package://xpp_cyberdog/meshes/link_knee_fr.STL; visual mesh filename=package://xpp_cyberdog/meshes/link_knee_fr.STL
- link FR_hip: geometry collision mesh filename=package://xpp_cyberdog/meshes/link_abad_fr.STL; visual mesh filename=package://xpp_cyberdog/meshes/link_abad_fr.STL
- link FR_thigh: geometry collision mesh filename=package://xpp_cyberdog/meshes/link_hip_fr.STL; visual mesh filename=package://xpp_cyberdog/meshes/link_hip_fr.STL
- link RL_calf: geometry collision mesh filename=package://xpp_cyberdog/meshes/link_knee_bl.STL; visual mesh filename=package://xpp_cyberdog/meshes/link_knee_bl.STL
- link RL_hip: geometry collision mesh filename=package://xpp_cyberdog/meshes/link_abad_bl.STL; visual mesh filename=package://xpp_cyberdog/meshes/link_abad_bl.STL
- link RL_thigh: geometry collision mesh filename=package://xpp_cyberdog/meshes/link_hip_bl.STL; visual mesh filename=package://xpp_cyberdog/meshes/link_hip_bl.STL
- link RR_calf: geometry collision mesh filename=package://xpp_cyberdog/meshes/link_knee_br.STL; visual mesh filename=package://xpp_cyberdog/meshes/link_knee_br.STL
- link RR_hip: geometry collision mesh filename=package://xpp_cyberdog/meshes/link_abad_br.STL; visual mesh filename=package://xpp_cyberdog/meshes/link_abad_br.STL
- link RR_thigh: geometry collision mesh filename=package://xpp_cyberdog/meshes/link_hip_br.STL; visual mesh filename=package://xpp_cyberdog/meshes/link_hip_br.STL
- link trunk: geometry collision mesh filename=package://xpp_cyberdog/meshes/body.STL; visual mesh filename=package://xpp_cyberdog/meshes/body.STL
